File: kicad/arduinowalkietalkie.sch (KiCad schematic (older format))
At the start: 31 parts, among them SW1 SW_Push_Dual, SW10 SW_Push_Dual, SW11 SW_Push_Dual, SW12 SW_Push_Dual, SW13 SW_Push_Dual, SW14 SW_Push_Dual, SW2 SW_Push_Dual, SW3 SW_Push_Dual, SW4 SW_Push_Dual, SW5 SW_Push_Dual, SW6 SW_Push_Dual, SW7 SW_Push_Dual, SW8 SW_Push_Dual, SW9 SW_Push_Dual, U1 NRF24L01_Breakout

Commit message: gerber file
Parts:
- added BZ1: Buzzer, BUZZER:BUZZER, symbol Device:Buzzer
- BMP1: footprint (none) -> BMP280:BMP280
- BT1: footprint (none) -> BAT_LIION_3V7:BAT_LIION_3V7
- CC1: footprint (none) -> DD05CVSA:DD05CVSA
- JP1: footprint (none) -> PIN_JUMPER:PIN_JUMPER
- R1, R2, R3, R4, R5, R6, R7, R8, R9: footprint (none) -> Resistor_THT:R_Axial_DIN0207_L6.3mm_D2.5mm_P7.62mm_Horizontal
- SW1, SW10, SW11, SW12, SW13, SW14, SW2, SW3, SW4, SW5, SW6, SW7, SW8, SW9: footprint (none) -> Button_Switch_THT:SW_TH_Tactile_Omron_B3F-10xx
- TFT1: footprint (none) -> TFT_KMR_18_SPI:TFT_KMR_1.8_SPI
Connections:
- net GND: now also BZ1.2 (+)
- net at A1.7 (D4): now also BZ1.1 (-)
- no-connect marks 43 -> 42
Other:
- note removed: "1"
- note removed: "8. 2. 2019"
- note removed: "Arduino Walkie Talkie"
Changed lines of the file:
@@
 EESchema Schematic File Version 4
+LIBS:arduinowalkietalkie-cache
 EELAYER 26 0
 EELAYER END
@@
 encoding utf-8
 Sheet 1 1
-Title ""
-Date ""
-Rev ""
+Title "Arduino Walkie Talkie"
+Date "2019-02-08"
+Rev "1"
 Comp ""
 Comment1 ""
 Comment2 ""
-Comment3 ""
-Comment4 ""
+Comment3 "License: Beerware rev42"
+Comment4 "Author: Lenart Arvo Kos"
 $EndDescr
 $Comp
@@
 F 0 "SW2" H 2750 4485 50  0000 C CNN
 F 1 "SW_Push_Dual" H 2750 4394 50  0000 C CNN
-F 2 "" H 2750 4400 50  0001 C CNN
+F 2 "Button_Switch_THT:SW_TH_Tactile_Omron_B3F-10xx" H 2750 4400 50  0001 C CNN
 F 3 "" H 2750 4400 50  0001 C CNN
 	1    2750 4200
@@
 F 0 "SW6" H 3350 4485 50  0000 C CNN
 F 1 "SW_Push_Dual" H 3350 4394 50  0000 C CNN
-F 2 "" H 3350 4400 50  0001 C CNN
+F 2 "Button_Switch_THT:SW_TH_Tactile_Omron_B3F-10xx" H 3350 4400 50  0001 C CNN
 F 3 "" H 3350 4400 50  0001 C CNN
 	1    3350 4200
@@
 F 0 "SW11" H 3950 4485 50  0000 C CNN
 F 1 "SW_Push_Dual" H 3950 4394 50  0000 C CNN
-F 2 "" H 3950 4400 50  0001 C CNN
+F 2 "Button_Switch_THT:SW_TH_Tactile_Omron_B3F-10xx" H 3950 4400 50  0001 C CNN
 F 3 "" H 3950 4400 50  0001 C CNN
 	1    3950 4200
@@
 F 0 "SW3" H 2750 5085 50  0000 C CNN
 F 1 "SW_Push_Dual" H 2750 4994 50  0000 C CNN
-F 2 "" H 2750 5000 50  0001 C CNN
+F 2 "Button_Switch_THT:SW_TH_Tactile_Omron_B3F-10xx" H 2750 5000 50  0001 C CNN
 F 3 "" H 2750 5000 50  0001 C CNN
 	1    2750 4800
@@
 F 0 "SW7" H 3350 5085 50  0000 C CNN
 F 1 "SW_Push_Dual" H 3350 4994 50  0000 C CNN
-F 2 "" H 3350 5000 50  0001 C CNN
+F 2 "Button_Switch_THT:SW_TH_Tactile_Omron_B3F-10xx" H 3350 5000 50  0001 C CNN
 F 3 "" H 3350 5000 50  0001 C CNN
 	1    3350 4800
@@
 F 0 "SW12" H 3950 5085 50  0000 C CNN
 F 1 "SW_Push_Dual" H 3950 4994 50  0000 C CNN
-F 2 "" H 3950 5000 50  0001 C CNN
+F 2 "Button_Switch_THT:SW_TH_Tactile_Omron_B3F-10xx" H 3950 5000 50  0001 C CNN
 F 3 "" H 3950 5000 50  0001 C CNN
 	1    3950 4800
@@
 F 0 "SW4" H 2750 5685 50  0000 C CNN
 F 1 "SW_Push_Dual" H 2750 5594 50  0000 C CNN
-F 2 "" H 2750 5600 50  0001 C CNN
+F 2 "Button_Switch_THT:SW_TH_Tactile_Omron_B3F-10xx" H 2750 5600 50  0001 C CNN
 F 3 "" H 2750 5600 50  0001 C CNN
 	1    2750 5400
@@
 F 0 "SW8" H 3350 5685 50  0000 C CNN
 F 1 "SW_Push_Dual" H 3350 5594 50  0000 C CNN
-F 2 "" H 3350 5600 50  0001 C CNN
+F 2 "Button_Switch_THT:SW_TH_Tactile_Omron_B3F-10xx" H 3350 5600 50  0001 C CNN
 F 3 "" H 3350 5600 50  0001 C CNN
 	1    3350 5400
@@
 F 0 "SW13" H 3950 5685 50  0000 C CNN
 F 1 "SW_Push_Dual" H 3950 5594 50  0000 C CNN
-F 2 "" H 3950 5600 50  0001 C CNN
+F 2 "Button_Switch_THT:SW_TH_Tactile_Omron_B3F-10xx" H 3950 5600 50  0001 C CNN
 F 3 "" H 3950 5600 50  0001 C CNN
 	1    3950 5400
@@
 F 0 "SW5" H 2750 6285 50  0000 C CNN
 F 1 "SW_Push_Dual" H 2750 6194 50  0000 C CNN
-F 2 "" H 2750 6200 50  0001 C CNN
+F 2 "Button_Switch_THT:SW_TH_Tactile_Omron_B3F-10xx" H 2750 6200 50  0001 C CNN
 F 3 "" H 2750 6200 50  0001 C CNN
 	1    2750 6000
@@
 F 0 "SW9" H 3350 6285 50  0000 C CNN
 F 1 "SW_Push_Dual" H 3350 6194 50  0000 C CNN
-F 2 "" H 3350 6200 50  0001 C CNN
+F 2 "Button_Switch_THT:SW_TH_Tactile_Omron_B3F-10xx" H 3350 6200 50  0001 C CNN
 F 3 "" H 3350 6200 50  0001 C CNN
 	1    3350 6000
@@
 F 0 "SW14" H 3950 6285 50  0000 C CNN
 F 1 "SW_Push_Dual" H 3950 6194 50  0000 C CNN
-F 2 "" H 3950 6200 50  0001 C CNN
+F 2 "Button_Switch_THT:SW_TH_Tactile_Omron_B3F-10xx" H 3950 6200 50  0001 C CNN
 F 3 "" H 3950 6200 50  0001 C CNN
 	1    3950 6000
@@
 F 0 "R7" V 3857 3850 50  0000 C CNN
 F 1 "2k2" V 3766 3850 50  0000 C CNN
-F 2 "" V 3580 3850 50  0001 C CNN
+F 2 "Resistor_THT:R_Axial_DIN0207_L6.3mm_D2.5mm_P7.62mm_Horizontal" V 3580 3850 50  0001 C CNN
 F 3 "~" H 3650 3850 50  0001 C CNN
 	1    3650 3850
@@
 F 0 "R5" V 2843 3850 50  0000 C CNN
 F 1 "4.7k" V 2934 3850 50  0000 C CNN
-F 2 "" V 2980 3850 50  0001 C CNN
+F 2 "Resistor_THT:R_Axial_DIN0207_L6.3mm_D2.5mm_P7.62mm_Horizontal" V 2980 3850 50  0001 C CNN
 F 3 "~" H 3050 3850 50  0001 C CNN
 	1    3050 3850
@@
 F 0 "R2" H 2370 4646 50  0000 L CNN
 F 1 "15k" H 2370 4555 50  0000 L CNN
-F 2 "" V 2230 4600 50  0001 C CNN
+F 2 "Resistor_THT:R_Axial_DIN0207_L6.3mm_D2.5mm_P7.62mm_Horizontal" V 2230 4600 50  0001 C CNN
 F 3 "~" H 2300 4600 50  0001 C CNN
 	1    2300 4600
@@
 F 0 "R3" H 2370 5246 50  0000 L CNN
 F 1 "1k5" H 2370 5155 50  0000 L CNN
-F 2 "" V 2230 5200 50  0001 C CNN
+F 2 "Resistor_THT:R_Axial_DIN0207_L6.3mm_D2.5mm_P7.62mm_Horizontal" V 2230 5200 50  0001 C CNN
 F 3 "~" H 2300 5200 50  0001 C CNN
 	1    2300 5200
@@
 F 0 "R4" H 2370 5846 50  0000 L CNN
 F 1 "1k5" H 2370 5755 50  0000 L CNN
-F 2 "" V 2230 5800 50  0001 C CNN
+F 2 "Resistor_THT:R_Axial_DIN0207_L6.3mm_D2.5mm_P7.62mm_Horizontal" V 2230 5800 50  0001 C CNN
 F 3 "~" H 2300 5800 50  0001 C CNN
 	1    2300 5800
@@
 F 0 "R8" H 4520 5896 50  0000 L CNN
 F 1 "10k" H 4520 5805 50  0000 L CNN
-F 2 "" V 4380 5850 50  0001 C CNN
+F 2 "Resistor_THT:R_Axial_DIN0207_L6.3mm_D2.5mm_P7.62mm_Horizontal" V 4380 5850 50  0001 C CNN
 F 3 "~" H 4450 5850 50  0001 C CNN
 	1    4450 5850
@@
 F 0 "TFT1" H 8777 3146 50  0000 L CNN
 F 1 "1.8_SPI_TFT_128*160" H 8777 3055 50  0000 L CNN
-F 2 "" H 7300 3850 50  0001 C CNN
+F 2 "TFT_KMR_18_SPI:TFT_KMR_1.8_SPI" H 7300 3850 50  0001 C CNN
 F 3 "" H 7300 3850 50  0001 C CNN
 	1    7300 3850
@@
 Wire Wire Line
 	4450 6250 6700 6250
-Text Notes 9050 6900 2    118  ~ 0
-Arduino Walkie Talkie
-Text Notes 8450 7650 2    39   ~ 0
-8. 2. 2019
 $Comp
 L power:+5V #PWR010
@@
 	1    0    0    -1
 $EndComp
-Text Notes 10650 7650 2    39   ~ 0
-1
 $Comp
 L Switch:SW_Push_Dual SW1
@@
 F 0 "SW1" H 2750 3135 50  0000 C CNN
 F 1 "SW_Push_Dual" H 2750 3044 50  0000 C CNN
-F 2 "" H 2750 3050 50  0001 C CNN
+F 2 "Button_Switch_THT:SW_TH_Tactile_Omron_B3F-10xx" H 2750 3050 50  0001 C CNN
 F 3 "" H 2750 3050 50  0001 C CNN
 	1    2750 2850
@@
 F 0 "SW10" H 3950 3135 50  0000 C CNN
 F 1 "SW_Push_Dual" H 3950 3044 50  0000 C CNN
-F 2 "" H 3950 3050 50  0001 C CNN
+F 2 "Button_Switch_THT:SW_TH_Tactile_Omron_B3F-10xx" H 3950 3050 50  0001 C CNN
 F 3 "" H 3950 3050 50  0001 C CNN
 	1    3950 2850
@@
 F 0 "R6" H 3430 3154 50  0000 R CNN
 F 1 "10k" H 3430 3245 50  0000 R CNN
-F 2 "" V 3430 3200 50  0001 C CNN
+F 2 "Resistor_THT:R_Axial_DIN0207_L6.3mm_D2.5mm_P7.62mm_Horizontal" V 3430 3200 50  0001 C CNN
 F 3 "~" H 3500 3200 50  0001 C CNN
 	1    3500 3200
@@
 F 0 "R1" H 2320 3246 50  0000 L CNN
 F 1 "10k" H 2320 3155 50  0000 L CNN
-F 2 "" V 2180 3200 50  0001 C CNN
+F 2 "Resistor_THT:R_Axial_DIN0207_L6.3mm_D2.5mm_P7.62mm_Horizontal" V 2180 3200 50  0001 C CNN
 F 3 "~" H 2250 3200 50  0001 C CNN
 	1    2250 3200
@@
 F 0 "BT1" H 6558 3646 50  0000 L CNN
 F 1 "Battery" H 6558 3555 50  0000 L CNN
-F 2 "" V 6450 3660 50  0001 C CNN
+F 2 "BAT_LIION_3V7:BAT_LIION_3V7" V 6450 3660 50  0001 C CNN
 F 3 "~" V 6450 3660 50  0001 C CNN
 	1    6450 3600
@@
 F 0 "CC1" H 7378 2538 39  0000 L CNN
 F 1 "DD05CVSA" H 7378 2463 39  0000 L CNN
-F 2 "" H 6500 2800 39  0001 C CNN
+F 2 "DD05CVSA:DD05CVSA" H 6500 2800 39  0001 C CNN
 F 3 "" H 6500 2800 39  0001 C CNN
 	1    6800 2800
@@
 F 0 "JP1" H 7400 3814 50  0000 C CNN
 F 1 "Jumper" H 7400 3723 50  0000 C CNN
-F 2 "" H 7400 3550 50  0001 C CNN
+F 2 "PIN_JUMPER:PIN_JUMPER" H 7400 3550 50  0001 C CNN
 F 3 "~" H 7400 3550 50  0001 C CNN
 	1    7400 3550
@@
 F 0 "BMP1" H 3377 1638 39  0000 L CNN
 F 1 "BMP280" H 3377 1563 39  0000 L CNN
-F 2 "" H 2850 1800 39  0001 C CNN
+F 2 "BMP280:BMP280" H 2850 1800 39  0001 C CNN
 F 3 "" H 2850 1800 39  0001 C CNN
 	1    2850 1800
@@
 F 0 "R9" H 7020 4196 50  0000 L CNN
 F 1 "220" H 7020 4105 50  0000 L CNN
-F 2 "" V 6880 4150 50  0001 C CNN
+F 2 "Resistor_THT:R_Axial_DIN0207_L6.3mm_D2.5mm_P7.62mm_Horizontal" V 6880 4150 50  0001 C CNN
 F 3 "~" H 6950 4150 50  0001 C CNN
 	1    6950 4150
@@
 NoConn ~ 6200 4850
 NoConn ~ 6200 4450
-NoConn ~ 5200 4450
 NoConn ~ 5200 4150
 NoConn ~ 5200 4050
@@
 	1    0    0    -1
 $EndComp
+$Comp
+L Device:Buzzer BZ1
+U 1 1 5C5D1F9F
+P 4450 5100
+F 0 "BZ1" H 4456 4775 50  0000 C CNN
+F 1 "Buzzer" H 4456 4866 50  0000 C CNN
+F 2 "BUZZER:BUZZER" V 4425 5200 50  0001 C CNN
+F 3 "~" V 4425 5200 50  0001 C CNN
+	1    4450 5100
+	-1   0    0    1
+$EndComp
+Wire Wire Line
+	5200 4450 4700 4450
+Wire Wire Line
+	4700 4450 4700 5200
+Wire Wire Line
+	4700 5200 4550 5200
+$Comp
+L power:GND #PWR0101
+U 1 1 5C5D6BCF
+P 4600 5050
+F 0 "#PWR0101" H 4600 4800 50  0001 C CNN
+F 1 "GND" H 4605 4877 50  0000 C CNN
+F 2 "" H 4600 5050 50  0001 C CNN
+F 3 "" H 4600 5050 50  0001 C CNN
+	1    4600 5050
+	1    0    0    -1
+$EndComp
+Wire Wire Line
+	4550 5000 4600 5000
+Wire Wire Line
+	4600 5000 4600 5050
 $EndSCHEMATC

Commit message: update pcb
Parts:
- added JP2: Jumper, PIN_JUMPER:PIN_JUMPER, symbol Device:Jumper
- added R10, R11, R12, R13, R14: 2k7, Resistor_THT:R_Axial_DIN0207_L6.3mm_D2.5mm_P7.62mm_Horizontal, symbol Device:R
Connections:
- net MOSI: now also R12.2; no longer TFT1.9 (TFT_MOSI)
- net SCK: now also R11.2; no longer TFT1.8 (TFT_SCK)
- net at A1.11 (D8): now also R13.2; no longer TFT1.10 (TFT_DC)
- net at A1.12 (D9): now also R14.2; no longer TFT1.11 (TFT_RST)
- net at A1.13 (D10): now also R10.2; no longer TFT1.7 (TFT_CS)
- net at A1.27 (+5V): now also JP2.1; no longer CC1.1 (VIN)
- new net: R13.1, TFT1.10 (TFT_DC)
- new net: R14.1, TFT1.11 (TFT_RST)
- new net: R10.1, TFT1.7 (TFT_CS)
- new net: R11.1, TFT1.8 (TFT_SCK)
- new net: R12.1, TFT1.9 (TFT_MOSI)
- new net: CC1.1 (VIN), JP2.2
Other:
- moved on the sheet: TFT1
Changed lines of the file:
@@
 L TFT_KMR-1.8_SPI:1.8_SPI_TFT_128*160 TFT1
 U 1 1 5C5E391F
-P 7300 3850
-F 0 "TFT1" H 8777 3146 50  0000 L CNN
-F 1 "1.8_SPI_TFT_128*160" H 8777 3055 50  0000 L CNN
-F 2 "TFT_KMR_18_SPI:TFT_KMR_1.8_SPI" H 7300 3850 50  0001 C CNN
-F 3 "" H 7300 3850 50  0001 C CNN
-	1    7300 3850
+P 7700 3850
+F 0 "TFT1" H 9177 3146 50  0000 L CNN
+F 1 "1.8_SPI_TFT_128*160" H 9177 3055 50  0000 L CNN
+F 2 "TFT_KMR_18_SPI:TFT_KMR_1.8_SPI" H 7700 3850 50  0001 C CNN
+F 3 "" H 7700 3850 50  0001 C CNN
+	1    7700 3850
 	1    0    0    -1
 $EndComp
@@
 	1    0    0    -1
 $EndComp
-Wire Wire Line
-	7200 5400 7400 5400
 Text GLabel 5200 5150 0    50   Output ~ 0
 MOSI
@@
 	-1   0    0    1
 $EndComp
-Wire Wire Line
-	7200 3900 7400 3900
 Text GLabel 7400 4700 0    50   Input ~ 0
 MOSI
@@
 	5900 3650 5900 2850
 Wire Wire Line
-	5900 2850 6800 2850
+	5900 2850 6050 2850
 $Comp
 L power:GND #PWR012
@@
 $EndComp
 NoConn ~ 4700 3050
-NoConn ~ 7400 4100
-NoConn ~ 7400 4200
-NoConn ~ 7400 4300
-NoConn ~ 7400 4400
+NoConn ~ 7800 4100
+NoConn ~ 7800 4200
+NoConn ~ 7800 4300
+NoConn ~ 7800 4400
 NoConn ~ 2550 4200
 NoConn ~ 3150 4200
@@
 Wire Wire Line
 	6900 4300 6900 5300
-Wire Wire Line
-	6900 5300 7400 5300
 Connection ~ 5800 3550
 Wire Wire Line
 	5800 3550 5800 2100
-Wire Wire Line
-	7400 4000 6950 4000
 Wire Wire Line
 	6950 6100 4750 6100
@@
 Wire Wire Line
 	4600 5000 4600 5050
+$Comp
+L Device:R R10
+U 1 1 5C72199E
+P 7550 4500
+F 0 "R10" V 7343 4500 50  0000 C CNN
+F 1 "2k7" V 7434 4500 50  0000 C CNN
+F 2 "Resistor_THT:R_Axial_DIN0207_L6.3mm_D2.5mm_P7.62mm_Horizontal" V 7480 4500 50  0001 C CNN
+F 3 "~" H 7550 4500 50  0001 C CNN
+	1    7550 4500
+	0    1    1    0
+$EndComp
+Wire Wire Line
+	7700 4500 7800 4500
+Wire Wire Line
+	7700 4600 7750 4600
+Wire Wire Line
+	7700 4700 7800 4700
+Wire Wire Line
+	7800 4800 7700 4800
+Wire Wire Line
+	7700 4900 7800 4900
+Wire Wire Line
+	6900 5300 7800 5300
+Wire Wire Line
+	7200 5400 7800 5400
+Wire Wire Line
+	6950 4000 7800 4000
+Wire Wire Line
+	7200 3900 7800 3900
+$Comp
+L Device:R R11
+U 1 1 5C759F76
+P 7550 4600
+F 0 "R11" V 7343 4600 50  0000 C CNN
+F 1 "2k7" V 7434 4600 50  0000 C CNN
+F 2 "Resistor_THT:R_Axial_DIN0207_L6.3mm_D2.5mm_P7.62mm_Horizontal" V 7480 4600 50  0001 C CNN
+F 3 "~" H 7550 4600 50  0001 C CNN
+	1    7550 4600
+	0    1    1    0
+$EndComp
+Connection ~ 7750 4600
+Wire Wire Line
+	7750 4600 7800 4600
+$Comp
+L Device:R R12
+U 1 1 5C75A044
+P 7550 4700
+F 0 "R12" V 7343 4700 50  0000 C CNN
+F 1 "2k7" V 7434 4700 50  0000 C CNN
+F 2 "Resistor_THT:R_Axial_DIN0207_L6.3mm_D2.5mm_P7.62mm_Horizontal" V 7480 4700 50  0001 C CNN
+F 3 "~" H 7550 4700 50  0001 C CNN
+	1    7550 4700
+	0    1    1    0
+$EndComp
+$Comp
+L Device:R R13
+U 1 1 5C75A09A
+P 7550 4800
+F 0 "R13" V 7343 4800 50  0000 C CNN
+F 1 "2k7" V 7434 4800 50  0000 C CNN
+F 2 "Resistor_THT:R_Axial_DIN0207_L6.3mm_D2.5mm_P7.62mm_Horizontal" V 7480 4800 50  0001 C CNN
+F 3 "~" H 7550 4800 50  0001 C CNN
+	1    7550 4800
+	0    1    1    0
+$EndComp
+$Comp
+L Device:R R14
+U 1 1 5C75A0F2
+P 7550 4900
+F 0 "R14" V 7343 4900 50  0000 C CNN
+F 1 "2k7" V 7434 4900 50  0000 C CNN
+F 2 "Resistor_THT:R_Axial_DIN0207_L6.3mm_D2.5mm_P7.62mm_Horizontal" V 7480 4900 50  0001 C CNN
+F 3 "~" H 7550 4900 50  0001 C CNN
+	1    7550 4900
+	0    1    1    0
+$EndComp
+$Comp
+L Device:Jumper JP2
+U 1 1 5C75AD4F
+P 6350 2850
+F 0 "JP2" H 6350 3114 50  0000 C CNN
+F 1 "Jumper" H 6350 3023 50  0000 C CNN
+F 2 "PIN_JUMPER:PIN_JUMPER" H 6350 2850 50  0001 C CNN
+F 3 "~" H 6350 2850 50  0001 C CNN
+	1    6350 2850
+	1    0    0    -1
+$EndComp
+Wire Wire Line
+	6650 2850 6800 2850
 $EndSCHEMATC

Commit message: New pcb
Parts:
- added C1, C2, C3, C4: C, Capacitor_THT:C_Disc_D4.7mm_W2.5mm_P5.00mm, symbol Device:C
- added R15: 220, Resistor_THT:R_Axial_DIN0207_L6.3mm_D2.5mm_P7.62mm_Horizontal, symbol Device:R
- added R16: 10K, Resistor_THT:R_Axial_DIN0207_L6.3mm_D2.5mm_P7.62mm_Horizontal, symbol Device:R
- BMP1: symbol BMP280:BMP280 -> arduinowalkietalkie-rescue:BMP280-BMP280
- CC1: symbol DD05CVSA:DD05CVSA -> arduinowalkietalkie-rescue:DD05CVSA-DD05CVSA
- TFT1: symbol TFT_KMR-1.8_SPI:1.8_SPI_TFT_128*160 -> arduinowalkietalkie-rescue:1.8_SPI_TFT_128*160-TFT_KMR-1.8_SPI
Connections:
- wire segments 146 -> 156
- no-connect marks 42 -> 41
Other:
- moved on the sheet: BT1, BZ1, CC1, D1, JP1, JP2
